Commit message: Enhance FANUC LR Mate 200iC URDF model with improved joint limits, dimensions, and materials. Update curriculum training script to support GPU and parallel environments, add accuracy monitoring, and refine reward structure. Introduce domain randomization in RL environment and enhance robot simulation with better URDF loading and rendering capabilities.

File: res/fanuc_lrmate_200ic.urdf (robot description, URDF)
Before this commit: robot fanuc_lrmate_200ic, 8 links, 7 joints
Links:
- link base_link: mass 5.0 -> 7.0; geometry collision cylinder length=0.15 radius=0.12; visual cylinder length=0.15 radius=0.12
- link link_1: mass 4.8 -> 4.5; geometry collision cylinder length=0.12 radius=0.095; visual cylinder length=0.12 radius=0.095
- link link_2: geometry collision box size=0.12 0.19 0.12; visual box size=0.12 0.19 0.12
- link link_4: mass 2.0 -> 2.5; geometry collision cylinder length=0.085 radius=0.045; visual cylinder length=0.085 radius=0.045
- link link_5: mass 1.5 -> 2.0; geometry collision cylinder length=0.085 radius=0.045; visual cylinder length=0.085 radius=0.045
- link link_6: mass 0.5 -> 1.0
- link tool0: mass 0.001 -> 0.1; geometry collision cylinder length=0.01 radius=0.031; visual cylinder length=0.01 radius=0.031
Joints:
- joint joint_1: limit lower=-2.97 upper=2.97 effort=10 velocity=6.11 -> lower=-2.97 upper=2.97 effort=11.9 velocity=6.11; origin xyz=0 0 0.17 rpy=0 0 0 -> xyz=0 0 0.15 rpy=0 0 0
- joint joint_2: limit lower=-1.05 upper=2.18 effort=10 velocity=6.11 -> lower=-1.05 upper=2.44 effort=11.9 velocity=6.11; origin xyz=0.05 0 0.17 rpy=0 0 0 -> xyz=0.05 0 0.13 rpy=0 0 0
- joint joint_3: limit lower=-3.14 upper=1.22 effort=10 velocity=6.98 -> lower=-2.13 upper=4.64 effort=11.9 velocity=6.98; origin xyz=0.1 0 0 rpy=0 0 0 -> xyz=0.12 0 0 rpy=0 0 0
- joint joint_4: limit lower=-3.32 upper=3.32 effort=10 velocity=7.85 -> lower=-3.31 upper=3.31 effort=11.9 velocity=7.85
- joint joint_5: limit lower=-2.09 upper=2.09 effort=10 velocity=7.85 -> lower=-2.09 upper=2.09 effort=11.9 velocity=7.85; origin xyz=0 0 0.08 rpy=0 0 0 -> xyz=0 0 0.085 rpy=0 0 0
- joint joint_6: limit lower=-6.28 upper=6.28 effort=10 velocity=12.57 -> lower=-6.28 upper=6.28 effort=6.7 velocity=12.57; origin xyz=0 0 0.08 rpy=0 0 0 -> xyz=0 0 0.085 rpy=0 0 0
